File: pcb/ledboard/ledboard.sch (KiCad schematic (older format))
At the start: 30 parts, among them J1 LEFT, J2 PWR_L, J3 RIGHT, J4 PWR_R, U1 AL8860, U2 AL8860

Commit message: Created LED Board
Parts:
- removed D7: GRN, ledboard:LTST-S220, symbol Device:LED
- removed D8: RED, ledboard:LTST-S220, symbol Device:LED
- removed J1: LEFT, ledboard:PinHeader_1x02_P2.54mm_Vertical_RoundRect, symbol Connector_Generic:Conn_01x02
- removed J2: PWR_L, ledboard:PinHeader_1x02_P2.54mm_Vertical_RoundRect, symbol Connector_Generic:Conn_01x02
- removed J3: RIGHT, ledboard:PinHeader_1x02_P2.54mm_Vertical_RoundRect, symbol Connector_Generic:Conn_01x02
- removed J4: PWR_R, ledboard:PinHeader_1x02_P2.54mm_Vertical_RoundRect, symbol Connector_Generic:Conn_01x02
- removed R3, R4: 180, Resistor_SMD:R_0402_1005Metric, symbol Device:R
- removed R6, R7, R8: 47k, Resistor_SMD:R_0402_1005Metric, symbol Device:R_Small
- added J1: Conn_01x03, ledboard:WJ250B-3pin, symbol Connector_Generic:Conn_01x03
Connections:
- net labels added: CTRL
- net labels removed: CTRL_L, CTRL_R, USR_LED_A, USR_LED_B
- wire segments 99 -> 77
Other:
- moved on the sheet: R5

Commit message: Finished pcb
Parts:
- C3, C4: footprint Capacitor_SMD:C_0402_1005Metric -> Capacitor_SMD:C_0603_1608Metric
Changed lines of the file:
@@
 F 0 "C3" H 1408 2596 50  0000 R CNN
 F 1 "100n" H 1408 2505 50  0000 R CNN
-F 2 "Capacitor_SMD:C_0402_1005Metric" H 1538 2400 50  0001 C CNN
+F 2 "Capacitor_SMD:C_0603_1608Metric" H 1538 2400 50  0001 C CNN
 F 3 "~" H 1500 2550 50  0001 C CNN
 F 4 "CC0402KRX5R8BB104" H 1500 2550 50  0001 C CNN "P/N"
@@
 F 0 "C4" H 4608 2596 50  0000 R CNN
 F 1 "100n" H 4608 2505 50  0000 R CNN
-F 2 "Capacitor_SMD:C_0402_1005Metric" H 4738 2400 50  0001 C CNN
+F 2 "Capacitor_SMD:C_0603_1608Metric" H 4738 2400 50  0001 C CNN
 F 3 "~" H 4700 2550 50  0001 C CNN
 F 4 "CC0402KRX5R8BB104" H 4700 2550 50  0001 C CNN "P/N"

Commit message: ledboard kinda done???
Parts:
- added J2: Conn_01x02, Connector_AMASS:AMASS_XT30U-M_1x02_P5.0mm_Vertical, symbol Connector_Generic:Conn_01x02
- R5: footprint Resistor_SMD:R_0402_1005Metric -> Resistor_SMD:R_0603_1608Metric
Connections:
- net +12V: now also J2.2 (Pin_2)
- net GND: now also J2.1 (Pin_1)
Changed lines of the file:
@@
 F 0 "R5" H 1541 4496 50  0000 R CNN
 F 1 "47k" H 1541 4405 50  0000 R CNN
-F 2 "Resistor_SMD:R_0402_1005Metric" H 1600 4450 50  0001 C CNN
+F 2 "Resistor_SMD:R_0603_1608Metric" H 1600 4450 50  0001 C CNN
 F 3 "~" H 1600 4450 50  0001 C CNN
 F 4 "0402WGJ0473TCE" H 1600 4450 50  0001 C CNN "P/N"
@@
 	1800 4600 1800 4700
 Connection ~ 2350 4550
+$Comp
+L Connector_Generic:Conn_01x02 J2
+U 1 1 6243F974
+P 3200 4800
+F 0 "J2" H 3280 4792 50  0000 L CNN
+F 1 "Conn_01x02" H 3280 4701 50  0000 L CNN
+F 2 "Connector_AMASS:AMASS_XT30U-M_1x02_P5.0mm_Vertical" H 3200 4800 50  0001 C CNN
+F 3 "~" H 3200 4800 50  0001 C CNN
+	1    3200 4800
+	1    0    0    -1
+$EndComp
+Wire Wire Line
+	2350 4600 2350 4900
+Wire Wire Line
+	2350 4900 3000 4900
+Connection ~ 2350 4600
+Wire Wire Line
+	1650 4900 1650 4750
+Wire Wire Line
+	1650 4750 1250 4750
+Wire Wire Line
+	1250 4750 1250 4150
+Wire Wire Line
+	1250 4150 3000 4150
+Wire Wire Line
+	3000 4150 3000 4800
 $EndSCHEMATC
