File: pcb/ledboard/ledboard.kicad_pcb (KiCad board)
At the start: 2 copper layers, 105 x 78.5 mm, 20 parts, among them J1 Conn_01x03, U1 AL8860, U2 AL8860

Commit message: started v2
Parts:
- moved D6 112.1 mm to (202.0, 112.0), turned to 180 degrees
- moved J1 108.9 mm to (60.0, 129.0), turned to 0 degrees
- moved R5 102.3 mm to (138.9, 148.4), turned to 0 degrees
- moved D4 98.2 mm to (100.9, 134.2), turned to 270 degrees
- moved C5 96.2 mm to (97.9, 129.9), turned to 90 degrees
- moved C3 94.0 mm to (99.4, 129.9), turned to 90 degrees
- moved R2 93.0 mm to (103.9, 133.4), turned to 90 degrees
- moved C1 91.9 mm to (100.9, 129.9), turned to 90 degrees
- moved U2 86.3 mm to (103.9, 128.9), turned to 270 degrees
- moved L2 75.8 mm to (111.0, 128.0), turned to 180 degrees
- moved R1 72.0 mm to (99.9, 84.6), turned to 90 degrees
- moved D1 71.2 mm to (101.9, 81.1), turned to 0 degrees
- moved U1 66.3 mm to (102.9, 84.7), turned to 270 degrees
- moved C2 62.6 mm to (105.9, 82.8), turned to 90 degrees
- moved C4 60.6 mm to (107.4, 82.1), turned to 90 degrees
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Routing:
- net GND: track 315.7 -> 0.00 mm
- net /CTRL: track 295.0 -> 0.00 mm
- net +12V: track 186.5 -> 0.00 mm
- net Net-(D6-Pad1): track 60.5 -> 0.00 mm
- net Net-(D3-Pad1): track 51.8 -> 0.00 mm
- net Net-(D5-Pad1): track 41.4 -> 0.00 mm
- net Net-(D2-Pad1): track 41.4 -> 0.00 mm
- net Net-(D4-Pad2): track 25.6 -> 0.00 mm
- net Net-(D1-Pad2): track 21.6 -> 0.00 mm
- net Net-(D5-Pad2): track 17.0 -> 0.00 mm
- net Net-(D2-Pad2): track 7.00 -> 0.00 mm
- removed copper zone on F.Cu, net GND
Other:
- board size 105 x 78.5 mm -> 161 x 87 mm
- board text added: "LED Booster By Ethan Cao Rev. 2"
- board text removed: "LED Booster By Ethan Cao Rev. 1"

Commit message: ledboard kinda done???
Parts:
- added J2: Conn_01x02, Connector_AMASS:AMASS_XT30U-M_1x02_P5.0mm_Vertical, F.Cu at (70.0, 136.0)
- R5: footprint Resistor_SMD:R_0402_1005Metric -> Resistor_SMD:R_0603_1608Metric
- moved J1 140.0 mm to (200.0, 129.0)
- moved C5 113.7 mm to (192.0, 66.0), turned to 180 degrees
- moved D4 111.7 mm to (198.0, 79.0), turned to 90 degrees
- moved C1 109.6 mm to (192.0, 69.0), turned to 180 degrees
- moved C3 109.2 mm to (192.0, 72.0), turned to 180 degrees
- moved L2 105.1 mm to (192.0, 61.0)
- moved U2 101.2 mm to (192.0, 79.0)
- moved R2 100.0 mm to (192.0, 86.0), turned to 0 degrees
- moved R5 69.8 mm to (207.0, 133.0)
- moved L1 41.5 mm to (84.0, 61.0), turned to 0 degrees
- moved C6 34.4 mm to (84.0, 66.0), turned to 180 degrees
- moved C4 26.8 mm to (84.0, 69.0), turned to 180 degrees
- moved U1 25.5 mm to (78.0, 79.0)
- moved C2 24.4 mm to (84.0, 72.0), turned to 180 degrees
- moved R1 21.9 mm to (78.0, 86.0), turned to 0 degrees
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Routing:
- net GND: track 0.00 -> 443.3 mm
- net +12V: track 0.00 -> 410.6 mm
- net /CTRL: track 0.00 -> 199.7 mm
- net Net-(D5-Pad1): track 0.00 -> 108.9 mm
- net Net-(D2-Pad1): track 0.00 -> 107.4 mm
- net Net-(D3-Pad1): track 0.00 -> 58.8 mm
- net Net-(D6-Pad1): track 0.00 -> 55.8 mm
- net Net-(D5-Pad2): track 0.00 -> 45.2 mm
- net Net-(D2-Pad2): track 0.00 -> 44.4 mm
- net Net-(D1-Pad2): track 0.00 -> 23.7 mm
- net Net-(D4-Pad2): track 0.00 -> 23.0 mm
- net (no net): vias 4 -> 0
Other:
- outline, holes or cut-outs redrawn
- net class Power added: clearance 0.15, trace_width 2, via_dia 0.5, via_drill 0.25

Commit message: Update ledboard.kicad_pcb
Other:
- board size 161 x 87 mm -> 163 x 87 mm
Changed lines of the file:
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@@
     )
   )
-  (gr_circle (center 60.2 87) (end 62 87) (layer Edge.Cuts) (width 0.15))
-  (gr_circle (center 213 87) (end 214.8 87) (layer Edge.Cuts) (width 0.15))
-  (gr_circle (center 139 58) (end 140.8 58) (layer Edge.Cuts) (width 0.15))
-  (gr_circle (center 60.2 58) (end 62 58) (layer Edge.Cuts) (width 0.15))
-  (gr_circle (center 213 58) (end 214.8 58) (layer Edge.Cuts) (width 0.15))
+  (gr_circle (center 61 87) (end 62.8 87) (layer Edge.Cuts) (width 0.15))
+  (gr_circle (center 214 87) (end 215.8 87) (layer Edge.Cuts) (width 0.15))
+  (gr_circle (center 137.5 59) (end 139.3 59) (layer Edge.Cuts) (width 0.15))
+  (gr_circle (center 61 59) (end 62.8 59) (layer Edge.Cuts) (width 0.15))
+  (gr_circle (center 214 59) (end 215.8 59) (layer Edge.Cuts) (width 0.15))
   (gr_circle (center 93 135) (end 95.5 135) (layer Edge.Cuts) (width 0.15))
   (gr_circle (center 181.9 135) (end 184.4 135) (layer Edge.Cuts) (width 0.15))
@@
   (gr_line (start 177 129) (end 177 91.5) (layer Edge.Cuts) (width 0.15))
   (gr_arc (start 175 91.5) (end 177 91.5) (angle -90) (layer Edge.Cuts) (width 0.05))
-  (gr_line (start 217 59) (end 217 136) (layer Edge.Cuts) (width 0.05))
+  (gr_line (start 219 59) (end 219 136) (layer Edge.Cuts) (width 0.05))
   (gr_arc (start 100 91.5) (end 100 89.5) (angle -90) (layer Edge.Cuts) (width 0.05))
   (gr_line (start 98 91.5) (end 98 129) (layer Edge.Cuts) (width 0.15))
   (gr_arc (start 175 129) (end 175 131) (angle -90) (layer Edge.Cuts) (width 0.05))
-  (gr_arc (start 212 136) (end 212 141) (angle -90) (layer Edge.Cuts) (width 0.05))
+  (gr_arc (start 214 136) (end 214 141) (angle -90) (layer Edge.Cuts) (width 0.05))
   (gr_line (start 100 131) (end 175 131) (layer Edge.Cuts) (width 0.15))
-  (gr_arc (start 212 59) (end 217 59) (angle -90) (layer Edge.Cuts) (width 0.05))
+  (gr_arc (start 214 59) (end 219 59) (angle -90) (layer Edge.Cuts) (width 0.05))
   (gr_line (start 100 89.5) (end 175 89.5) (layer Edge.Cuts) (width 0.15))
   (gr_arc (start 61 59) (end 61 54) (angle -90) (layer Edge.Cuts) (width 0.05))
-  (gr_line (start 212 141) (end 61 141) (layer Edge.Cuts) (width 0.05))
+  (gr_line (start 214 141) (end 61 141) (layer Edge.Cuts) (width 0.05))
   (gr_arc (start 100 129) (end 98 129) (angle -90) (layer Edge.Cuts) (width 0.05))
   (gr_arc (start 61 136) (end 56 136) (angle -90) (layer Edge.Cuts) (width 0.05))
-  (gr_line (start 61 54) (end 212 54) (layer Edge.Cuts) (width 0.05))
+  (gr_line (start 61 54) (end 214 54) (layer Edge.Cuts) (width 0.05))
   (segment (start 78.9375 83.1612) (end 78.9375 80.3225) (width 1) (layer F.Cu) (net 1))
   (segment (start 78.9375 80.3225) (end 78.95 80.31) (width 1) (layer F.Cu) (net 1))

Commit message: Update ledboard.kicad_pcb
Parts:
- moved C5 14.5 mm to (183.4, 77.7), turned to 90 degrees
- moved C1 10.4 mm to (186.3, 77.7), turned to 90 degrees
- moved C3 6.45 mm to (189.0, 77.7), turned to 90 degrees
Routing:
- net +12V: track 410.6 -> 427.3 mm
- net GND: track 443.3 -> 439.4 mm
- net Net-(D2-Pad2): track 44.4 -> 46.6 mm
- added copper zone on F.Cu, net GND

Commit message: Update ledboard.kicad_pcb
Routing:
- net +12V: track 427.3 -> 416.5 mm
- net GND: track 439.4 -> 440.5 mm
